Commit message: fixed launch/urdf files to load STL files w/o err

File: bazu/urdf/bazu_gazebo.urdf (robot description, URDF)
Before this commit: robot bazu, 8 links, 7 joints
Links:
- link base: geometry collision mesh filename=package://base.stl; visual mesh filename=package://base.stl
- link link_1: geometry collision mesh filename=package://joint_1.stl; visual mesh filename=package://joint_1.stl
- link link_2: geometry collision mesh filename=package://joint_2.stl; visual mesh filename=package://joint_2.stl
- link link_3: geometry collision mesh filename=package://joint_3.stl; visual mesh filename=package://joint_3.stl
- link link_4: geometry collision mesh filename=package://joint_4.stl; visual mesh filename=package://joint_4.stl
- link link_5: geometry collision mesh filename=package://joint_5.stl; visual mesh filename=package://joint_5.stl
- link link_6: geometry collision mesh filename=package://joint_6.stl; visual mesh filename=package://joint_6.stl
